File: nixie_board/nixie_board.kicad_pcb (KiCad board)
At the start: 2 copper layers, 221 x 59.7 mm, 53 parts, among them J1 12V, J2 170V, J3 GND, J4 SHTDWN, U1 74LS32, U10 74LS32, U11 K155NA1, U12 L7805, U13 74HCT595, U14 K155NA1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

Commit message: rev 0.2
Parts:
- added C15: 10uF, Capacitor_THT:CP_Radial_D5.0mm_P2.00mm, B.Cu at (184.2, 50.8)
- added R9: 4.7K, Resistor_THT:R_Axial_DIN0207_L6.3mm_D2.5mm_P7.62mm_Horizontal, B.Cu at (47.0, 26.7)
- J1, J2, J3: moved to B.Cu
- J4: value SHTDWN -> SHDN; moved to B.Cu
- R7: moved to F.Cu
- U3: value ESP32 -> WeMos_D1_mini; footprint ESP32-DEVKITC-32D:MODULE_ESP32-DEVKITC-32D -> Module:WEMOS_D1_mini_light; moved to B.Cu
- moved R7 134.7 mm to (54.6, 34.3)
- moved C8 120.7 mm to (125.7, 50.8), turned to 90 degrees
- moved U15 75.4 mm to (66.0, 26.7)
- moved J1 24.6 mm to (252.7, 50.8), turned to 270 degrees
- moved J4 23.6 mm to (252.7, 61.0), turned to 270 degrees
- moved J3 22.7 mm to (252.7, 55.9), turned to 270 degrees
- moved U1 15.9 mm to (88.9, 31.8), turned to 90 degrees
- moved U10 15.9 mm to (205.7, 31.8), turned to 90 degrees
- moved U3 12.7 mm to (44.5, 57.1)
- moved R1 8.13 mm to (88.9, 69.8), turned to 45 degrees
- moved R8 8.13 mm to (68.6, 69.8), turned to 45 degrees
- moved R2 8.13 mm to (114.3, 69.8), turned to 45 degrees
- moved R6 8.13 mm to (231.1, 69.8), turned to 45 degrees
- moved C7 7.73 mm to (243.8, 53.3)
- moved R3 7.18 mm to (146.1, 69.8), turned to 45 degrees
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Connections:
- U15 pad 2: Net-(U15-Pad2) -> Net-(R9-Pad2)
- U3 pad 1: /3.3V -> (no net)
- U3 pad 10: (no net) -> GND
- U3 pad 11: (no net) -> /RCLK
- U3 pad 12: (no net) -> /SER
- U3 pad 13: (no net) -> Net-(R9-Pad2)
- U3 pad 14: GND -> (no net)
- U3 pad 2: (no net) -> Net-(R7-Pad2)
- U3 pad 4: (no net) -> /SRCLK
- U3 pad 5: (no net) -> /SHUTDOWN
- U3 pad 6: (no net) -> /RGB
- U3 pad 7: (no net) -> /STROBE
- U3 pad 8: (no net) -> /3.3V
- U3 pad 9: (no net) -> /5V
Other:
- board size 221 x 59.7 mm -> 215.9 x 53.3 mm
- net class 5v rail: clearance 0.25 -> 0.35; trace_width 0.28 -> 0.35
- net class Default: clearance 0.25 -> 0.3; trace_width 0.25 -> 0.3
- net class HighVoltage: trace_width 0.35 -> 0.5
- rule trace_clearance: 0.25 -> 0.3

Commit message: clearence review
Routing:
- net GND: track 0.00 -> 461.9 mm
- net /5V: track 0.00 -> 407.3 mm
- net /STROBE: track 0.00 -> 224.0 mm
- net /SHUTDOWN: track 0.00 -> 218.7 mm
- net /SRCLK: track 0.00 -> 204.0 mm, vias 0 -> 1
- net /RCLK: track 0.00 -> 177.4 mm
- net /170V: track 0.00 -> 157.5 mm
- net Net-(U10-Pad8): track 0.00 -> 56.5 mm
- net Net-(U1-Pad11): track 0.00 -> 56.0 mm, vias 0 -> 1
- net /SER: track 0.00 -> 51.4 mm
- net Net-(U6-Pad11): track 0.00 -> 51.2 mm
- net Net-(U11-Pad3): track 0.00 -> 49.1 mm
- net Net-(U13-Pad14): track 0.00 -> 48.2 mm
- net Net-(U4-Pad9): track 0.00 -> 47.4 mm
- net Net-(N3-Pad2): track 0.00 -> 44.6 mm
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Other:
- net class 5v rail: trace_width 0.35 -> 0.4
- net class Default: clearance 0.3 -> 0.254; trace_width 0.3 -> 0.254
- net class HighVoltage removed
- net class HighVoltageIN added: clearance 0.35, trace_width 0.5, via_dia 0.8, via_drill 0.4
- net class HighVoltageOut added: clearance 0.35, trace_width 0.4, via_dia 0.8, via_drill 0.4
- rule trace_clearance: 0.3 -> 0.254

Commit message: board review 3
Parts:
- added M1: MountingHole_3.2mm_M3, MountingHole:MountingHole_3.2mm_M3, F.Cu at (54.6, 24.1)
- added M2: MountingHole_3.2mm_M3, MountingHole:MountingHole_3.2mm_M3, F.Cu at (252.7, 24.1)
- added M3: MountingHole_3.2mm_M3, MountingHole:MountingHole_3.2mm_M3, F.Cu at (252.7, 69.8)
- added M4: MountingHole_3.2mm_M3, MountingHole:MountingHole_3.2mm_M3, F.Cu at (54.6, 69.8)
- added S1: Symbol_Highvoltage_Type1_CopperTop_Small, Symbol:Symbol_Highvoltage_Type1_CopperTop_Small, B.Cu at (241.3, 68.6)
- added S10: LOGO, Symbol:tube_silk, B.Cu at (166.4, 57.1)
- added S11: LOGO, Symbol:tube_silk, B.Cu at (199.4, 57.1)
- added S12: LOGO, Symbol:tube_silk, B.Cu at (224.8, 57.1)
- added S13: LOGO, Symbol:tube, F.Cu at (47.0, 68.6)
- added S14: LOGO, Symbol:nixie_clock, F.Cu at (55.9, 47.0)
- added S2: Symbol_HighVoltage_Type2_CopperTop_VerySmall, Symbol:Symbol_HighVoltage_Type2_CopperTop_VerySmall, F.Cu at (248.9, 38.1)
- added S3: OSHW-Symbol_6.7x6mm_Copper, Symbol:OSHW-Symbol_6.7x6mm_Copper, B.Cu at (45.7, 69.8)
- added S6: LOGO, Symbol:tube, F.Cu at (63.5, 68.6)
- added S7: LOGO, Symbol:tube_silk, B.Cu at (82.5, 57.1)
- added S8: LOGO, Symbol:tube_silk, B.Cu at (108.0, 57.1)
- added S9: LOGO, Symbol:tube_silk, B.Cu at (141.0, 57.1)
- moved R9 13.7 mm to (52.1, 39.4)
- moved R7 13.5 mm to (44.5, 25.4)
- moved C14 6.35 mm to (237.5, 59.7), turned to 90 degrees
- moved R8 5.39 mm to (72.4, 66.0), turned to 315 degrees
- moved J1 3.81 mm to (252.7, 54.6)
- moved U12 3.81 mm to (251.5, 48.3)
- moved J3 2.54 mm to (252.7, 58.4)
- moved R1 1.80 mm to (87.6, 71.1)
- moved R3 1.80 mm to (144.8, 71.1)
- moved R5 1.80 mm to (203.2, 71.1)
- moved C7 1.80 mm to (245.1, 54.6), turned to 270 degrees
- moved R2 1.80 mm to (113.0, 71.1)
- moved J2 1.80 mm to (245.1, 71.1)
- moved R4 1.80 mm to (170.2, 71.1)
- moved R6 1.80 mm to (229.9, 71.1)
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Connections:
- C7 pad 1: /5V -> Net-(C7-Pad1)
- D6 pad 2: (no net) -> Net-(D6-Pad2)
- J1 pad 1: Net-(J1-Pad1) -> Net-(C7-Pad1)
- N1 pad LHDP: (no net) -> Net-(N1-PadLHDP)
- N1 pad RHDP: (no net) -> Net-(N1-PadRHDP)
- N2 pad LHDP: (no net) -> Net-(N2-PadLHDP)
- N2 pad RHDP: (no net) -> Net-(N2-PadRHDP)
- N3 pad LHDP: (no net) -> Net-(N3-PadLHDP)
- N3 pad RHDP: (no net) -> Net-(N3-PadRHDP)
- N4 pad LHDP: (no net) -> Net-(N4-PadLHDP)
- N4 pad RHDP: (no net) -> Net-(N4-PadRHDP)
- N5 pad LHDP: (no net) -> Net-(N5-PadLHDP)
- N5 pad RHDP: (no net) -> Net-(N5-PadRHDP)
- N6 pad LHDP: (no net) -> Net-(N6-PadLHDP)
- N6 pad RHDP: (no net) -> Net-(N6-PadRHDP)
- U12 pad 1: Net-(J1-Pad1) -> Net-(C7-Pad1)
- U13 pad 9: (no net) -> Net-(U13-Pad9)
- U3 pad 1: (no net) -> Net-(U3-Pad1)
- U3 pad 14: (no net) -> Net-(U3-Pad14)
- U3 pad 15: (no net) -> Net-(U3-Pad15)
- U3 pad 16: (no net) -> Net-(U3-Pad16)
- U3 pad 3: (no net) -> Net-(U3-Pad3)
Routing:
- net Net-(U6-Pad8): track 41.0 -> 56.7 mm, vias 1 -> 0
- net Net-(U1-Pad11): track 56.0 -> 40.8 mm
- net Net-(C7-Pad1): track 0.00 -> 14.5 mm
- net Net-(U11-Pad3): track 49.1 -> 35.5 mm
- net Net-(U2-Pad6): track 34.7 -> 23.6 mm
- net Net-(U6-Pad11): track 51.2 -> 42.3 mm, vias 0 -> 1
- net Net-(N2-Pad2): track 35.9 -> 43.4 mm
- net Net-(R9-Pad2): track 36.8 -> 29.7 mm
- net Net-(J1-Pad1): track 6.88 -> 0.00 mm
- net Net-(N5-Pad1): track 24.0 -> 17.3 mm
- net /3.3V: track 33.8 -> 40.3 mm
- net Net-(R7-Pad2): track 26.2 -> 32.5 mm
- net /STROBE: track 224.0 -> 217.8 mm
- net Net-(U11-Pad6): track 29.7 -> 23.5 mm, vias 1 -> 0
- net Net-(U13-Pad7): track 18.2 -> 24.0 mm
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- added copper zone on B.Cu, net GND
- added copper zone on F.Cu, net GND
Other:
- board text added: "Federico Scozzafava Carlos Abad Sanchez"
- board text added: "Smart Nixie Clock"
- board text added: "github.com/vascofazza/smart_nixie_clock"

Commit message: final board review
Parts:
- added C16: 10uF, Capacitor_THT:CP_Radial_D5.0mm_P2.00mm, B.Cu at (66.0, 26.7)
- added C17: 10uF, Capacitor_THT:CP_Radial_D5.0mm_P2.00mm, B.Cu at (248.9, 66.0)
- added J5: Barrel_Jack_Switch, Connector_BarrelJack:BarrelJack_Horizontal, B.Cu at (251.5, 35.6)
- R7: moved to B.Cu
- moved R7 45.6 mm to (57.0, 69.2), turned to 180 degrees
- moved C7 25.2 mm to (261.7, 35.6), turned to 0 degrees
- moved S3 24.4 mm to (70.0, 67.7)
- moved R8 22.8 mm to (51.4, 57.1), turned to 0 degrees
- moved J2 21.0 mm to (264.2, 62.2), turned to 270 degrees
- moved S1 19.1 mm to (260.2, 65.7), turned to 270 degrees
- moved C8 15.6 mm to (122.6, 66.0), turned to 0 degrees
- moved C15 15.2 mm to (184.2, 66.0), turned to 0 degrees
- moved S2 14.2 mm to (251.5, 52.1)
- moved J1 13.7 mm to (264.2, 47.0)
- moved J3 13.1 mm to (264.2, 52.1)
- moved J4 12.5 mm to (264.2, 57.1)
- moved U12 11.7 mm to (254.0, 59.7)
- moved M2 11.5 mm to (264.2, 25.4)
- moved M3 11.5 mm to (264.2, 68.6)
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Connections:
- U1 pad 14: (no net) -> /5V
- U1 pad 7: (no net) -> GND
- U10 pad 14: (no net) -> /5V
- U10 pad 7: (no net) -> GND
- U3 pad 14: Net-(U3-Pad14) -> /STROBE
- U3 pad 7: /STROBE -> Net-(U3-Pad7)
- U6 pad 14: (no net) -> /5V
- U6 pad 7: (no net) -> GND
Routing:
- net GND: track 467.4 -> 6.02 mm, vias 0 -> 11
- net /5V: track 411.9 -> 502.0 mm
- net /SHUTDOWN: track 219.2 -> 245.8 mm
- net /170V: track 157.5 -> 183.6 mm
- net Net-(C7-Pad1): track 14.5 -> 39.6 mm
- net /RGB: track 40.9 -> 15.9 mm
- net Net-(R7-Pad2): track 32.5 -> 18.6 mm
- net Net-(U1-Pad11): track 40.8 -> 54.4 mm, vias 1 -> 0
- net /3.3V: track 40.3 -> 53.5 mm
- net Net-(U1-Pad10): track 29.8 -> 42.3 mm
- net /STROBE: track 217.8 -> 206.0 mm
- net Net-(U6-Pad11): track 42.3 -> 52.7 mm
- net Net-(N1-Pad0): track 30.5 -> 21.8 mm
- net Net-(N4-Pad8): track 35.0 -> 26.4 mm
- net Net-(U10-Pad11): track 42.3 -> 50.7 mm
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Other:
- board size 215.9 x 53.3 mm -> 227.3 x 50.8 mm
- net class 5v rail: clearance 0.35 -> 0.254; trace_width 0.4 -> 0.3
- net class HighVoltageOut: clearance 0.35 -> 0.3
- board text added: "CroNixie Tube Clock"
- board text added: "Federico Scozzafava Carlos Abad Sánchez"
- board text added: "JLCJLCJLCJLC"
- board text removed: "Federico Scozzafava Carlos Abad Sanchez"
- board text removed: "Smart Nixie Clock"

Commit message: PCB version 2
Parts:
- added JP1: Jumper_3_Bridged12, Connector_Wire:SolderWirePad_1x03_P3.175mm_Drill1mm, B.Cu at (242.6, 40.6)
- added NL1: IN-3, nixies-us:nixies-us-IN-3, F.Cu at (123.6, 52.1)
- added NR1: IN-3, nixies-us:nixies-us-IN-3, F.Cu at (185.1, 52.1)
- added Q1: MPSA42, Package_TO_SOT_THT:TO-92_Wide, B.Cu at (256.5, 44.5)
- added Q2: MPSA42, Package_TO_SOT_THT:TO-92_Wide, B.Cu at (125.1, 44.5)
- added Q3: MPSA42, Package_TO_SOT_THT:TO-92_Wide, B.Cu at (186.7, 44.5)
- added Q4: MPSA42, Package_TO_SOT_THT:TO-92_Wide, B.Cu at (248.9, 44.5)
- added R10: 10K, Resistor_THT:R_Axial_DIN0207_L6.3mm_D2.5mm_P7.62mm_Horizontal, B.Cu at (248.9, 48.3)
- added R11: 10K, Resistor_THT:R_Axial_DIN0207_L6.3mm_D2.5mm_P7.62mm_Horizontal, B.Cu at (124.5, 33.0)
- added R12: 10K, Resistor_THT:R_Axial_DIN0207_L6.3mm_D2.5mm_P7.62mm_Horizontal, B.Cu at (129.5, 41.9)
- added R13: 10K, Resistor_THT:R_Axial_DIN0207_L6.3mm_D2.5mm_P7.62mm_Horizontal, B.Cu at (182.9, 33.0)
- added R14: 10K, Resistor_THT:R_Axial_DIN0207_L6.3mm_D2.5mm_P7.62mm_Horizontal, B.Cu at (191.1, 41.9)
- added R15: 100K, Resistor_THT:R_Axial_DIN0207_L6.3mm_D2.5mm_P7.62mm_Horizontal, B.Cu at (242.6, 45.7)
- U15: footprint Package_TO_SOT_THT:TO-92_Inline -> Package_TO_SOT_THT:TO-92_Inline_Wide
- moved U2 44.4 mm to (90.2, 78.7), turned to 90 degrees
- moved U7 44.4 mm to (148.6, 78.7), turned to 90 degrees
- moved U5 44.1 mm to (118.7, 78.7), turned to 90 degrees
- moved U11 44.0 mm to (207.6, 78.1), turned to 90 degrees
- moved U14 44.0 mm to (236.9, 78.1), turned to 90 degrees
- moved U9 43.8 mm to (177.8, 78.1), turned to 90 degrees
- moved C3 38.1 mm to (124.5, 77.5), turned to 90 degrees
- moved C4 38.1 mm to (154.3, 77.5), turned to 90 degrees
- moved C5 38.1 mm to (183.5, 77.5), turned to 90 degrees
- moved C6 37.9 mm to (95.9, 77.4), turned to 90 degrees
- moved C2 37.5 mm to (213.4, 76.8), turned to 90 degrees
- moved C1 32.6 mm to (242.4, 72.1)
- moved R5 26.1 mm to (214.0, 45.1), turned to 135 degrees
- moved R4 26.1 mm to (156.2, 45.1), turned to 45 degrees
- moved R1 26.0 mm to (90.8, 45.1), turned to 135 degrees
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Connections:
- R1 pad 1: /170V -> Net-(JP1-Pad2)
- R2 pad 1: /170V -> Net-(JP1-Pad2)
- R3 pad 1: /170V -> Net-(JP1-Pad2)
- R4 pad 1: /170V -> Net-(JP1-Pad2)
- R5 pad 1: /170V -> Net-(JP1-Pad2)
- R6 pad 1: /170V -> Net-(JP1-Pad2)
- U3 pad 3: Net-(U3-Pad3) -> /LEFT_DOT
- U3 pad 7: Net-(U3-Pad7) -> /RIGHT_DOT
Routing:
- net GND: track 6.02 -> 628.2 mm, vias 11 -> 0
- net Net-(JP1-Pad2): track 0.00 -> 163.4 mm
- net /RIGHT_DOT: track 0.00 -> 151.1 mm
- net /170V: track 183.6 -> 40.4 mm
- net /LEFT_DOT: track 0.00 -> 104.1 mm
- net /5V: track 502.0 -> 600.8 mm
- net Net-(U7-Pad6): track 24.8 -> 95.5 mm
- net Net-(U2-Pad3): track 36.6 -> 106.6 mm
- net /STROBE: track 206.0 -> 271.4 mm
- net Net-(U8-Pad6): track 15.0 -> 79.5 mm
- net Net-(U7-Pad3): track 37.0 -> 99.5 mm
- net Net-(U6-Pad3): track 7.40 -> 61.8 mm
- net Net-(U11-Pad6): track 24.8 -> 74.4 mm
- net Net-(U4-Pad6): track 17.1 -> 65.9 mm
- net Net-(U13-Pad6): track 15.0 -> 63.4 mm
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Other:
- board size 227.3 x 50.8 mm -> 227.3 x 61 mm
- board text added: "Cloxie Tube Clock"
- board text added: "D"
- board text added: "Q"
- board text removed: "CroNixie Tube Clock"

Commit message: clearence review
Routing:
- net GND: track 628.2 -> 630.9 mm
