File: nixie_board/nixie_board.kicad_pcb (KiCad board)
At the start: 2 copper layers, 199.4 x 50.8 mm, 85 parts, among them J1 POWER, J5 Barrel_Jack_Switch, Q1 MPSA42, Q2 MPSA42, U1 74LS32, U10 74LS32, U11 K155ID1, U13 74HCT595, U14 K155ID1, U15 DS18B20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

Commit message: rev2 board
Parts:
- moved S2b 3.56 mm to (58.2, 52.7)
Routing:
- net GND: track 706.6 -> 713.5 mm
- net /3.3V: track 65.6 -> 64.3 mm
Changed lines of the file:
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@@
   (general
     (thickness 1.6)
-    (drawings 72)
-    (tracks 1363)
+    (drawings 115)
+    (tracks 1370)
     (zones 0)
     (modules 85)
@@
   (page A4)
   (layers
-    (0 F.Cu signal)
-    (31 B.Cu signal)
-    (32 B.Adhes user)
-    (33 F.Adhes user)
-    (34 B.Paste user)
-    (35 F.Paste user)
+    (0 F.Cu signal hide)
+    (31 B.Cu signal hide)
+    (32 B.Adhes user hide)
+    (33 F.Adhes user hide)
+    (34 B.Paste user hide)
+    (35 F.Paste user hide)
     (36 B.SilkS user)
     (37 F.SilkS user)
     (38 B.Mask user hide)
-    (39 F.Mask user)
+    (39 F.Mask user hide)
     (40 Dwgs.User user)
     (41 Cmts.User user hide)
@@
   )
   (module Symbol:OSHW-Symbol_6.7x6mm_Copper (layer B.Cu)
-    (at 54.61 52.705 90)
+    (at 58.166 52.705 90)
     (descr "Open Source Hardware Symbol")
     (tags "Logo Symbol OSHW")
@@
     )
   )
+  (gr_line (start 246.253 26.797) (end 236.982 26.797) (layer Dwgs.User) (width 0.15))
+  (gr_line (start 246.253 41.529) (end 246.253 26.797) (layer Dwgs.User) (width 0.15))
+  (gr_line (start 236.982 41.529) (end 246.253 41.529) (layer Dwgs.User) (width 0.15))
+  (gr_line (start 236.982 26.797) (end 236.982 41.529) (layer Dwgs.User) (width 0.15))
+  (gr_line (start 65.659 71.12) (end 68.329022 71.12) (layer Dwgs.User) (width 0.15))
+  (gr_line (start 65.659 71.12) (end 62.988978 71.12) (layer Dwgs.User) (width 0.15))
+  (gr_line (start 65.659 68.453) (end 65.659 73.787) (layer Dwgs.User) (width 0.15))
+  (gr_line (start 65.659 71.12) (end 65.659 68.453) (layer Dwgs.User) (width 0.15))
+  (gr_circle (center 65.659 71.12) (end 62.992 71.247) (layer Dwgs.User) (width 0.15))
+  (gr_line (start 228.6 52.07) (end 228.6 43.178078) (layer Dwgs.User) (width 0.15))
+  (gr_line (start 228.6 52.07) (end 237.491922 52.07) (layer Dwgs.User) (width 0.15))
+  (gr_line (start 228.6 52.07) (end 219.708078 52.07) (layer Dwgs.User) (width 0.15))
+  (gr_line (start 203.2 52.07) (end 203.2 43.168215) (layer Dwgs.User) (width 0.15))
+  (gr_line (start 203.2 52.07) (end 212.101785 52.07) (layer Dwgs.User) (width 0.15))
+  (gr_line (start 203.2 52.07) (end 194.298215 52.07) (layer Dwgs.User) (width 0.15))
+  (gr_line (start 167.005 52.07) (end 167.005 43.18697) (layer Dwgs.User) (width 0.15))
+  (gr_line (start 167.005 52.07) (end 175.895 52.07) (layer Dwgs.User) (width 0.15))
+  (gr_line (start 167.005 52.07) (end 158.12197 52.07) (layer Dwgs.User) (width 0.15))
+  (gr_line (start 105.41 52.07) (end 105.3846 43.248299) (layer Dwgs.User) (width 0.15))
+  (gr_line (start 105.3846 52.07) (end 96.562899 52.07) (layer Dwgs.User) (width 0.15))
+  (gr_line (start 105.41 52.07) (end 114.3 52.07) (layer Dwgs.User) (width 0.15))
+  (gr_line (start 80.01 52.07) (end 80.01 43.225474) (layer Dwgs.User) (width 0.15))
+  (gr_line (start 80.01 52.07) (end 88.854526 52.07) (layer Dwgs.User) (width 0.15))
+  (gr_line (start 141.605 52.07) (end 141.605 43.229742) (layer Dwgs.User) (width 0.15))
+  (gr_line (start 141.605 52.07) (end 150.445258 52.07) (layer Dwgs.User) (width 0.15))
+  (gr_line (start 141.605 52.07) (end 132.764742 52.07) (layer Dwgs.User) (width 0.15))
+  (gr_line (start 123.571 52.07) (end 123.571 54.966602) (layer Dwgs.User) (width 0.15))
+  (gr_line (start 123.571 52.07) (end 123.571 49.173398) (layer Dwgs.User) (width 0.15))
+  (gr_line (start 126.4666 52.07) (end 123.571 52.07) (layer Dwgs.User) (width 0.15))
+  (gr_line (start 123.571 52.07) (end 126.4666 52.07) (layer Dwgs.User) (width 0.15))
+  (gr_line (start 123.571 52.07) (end 120.674398 52.07) (layer Dwgs.User) (width 0.15))
+  (gr_line (start 185.1152 52.07) (end 185.1152 54.967381) (layer Dwgs.User) (width 0.15))
+  (gr_line (start 185.1152 52.07) (end 185.1152 49.172619) (layer Dwgs.User) (width 0.15))
+  (gr_line (start 185.1152 52.07) (end 188.012581 52.07) (layer Dwgs.User) (width 0.15))
+  (gr_line (start 185.1152 52.07) (end 182.217819 52.07) (layer Dwgs.User) (width 0.15))
+  (gr_line (start 56.515 73.66) (end 60.325 73.66) (layer Dwgs.User) (width 0.15))
+  (gr_line (start 58.42 71.755) (end 58.42 75.565) (layer Dwgs.User) (width 0.15))
+  (gr_line (start 58.42 28.575) (end 58.42 32.385) (layer Dwgs.User) (width 0.15))
+  (gr_line (start 56.515 30.48) (end 60.325 30.48) (layer Dwgs.User) (width 0.15))
+  (gr_line (start 248.285 30.48) (end 252.095 30.48) (layer Dwgs.User) (width 0.15))
+  (gr_line (start 250.19 28.575) (end 250.19 32.385) (layer Dwgs.User) (width 0.15))
+  (gr_line (start 250.19 71.755) (end 250.19 75.565) (layer Dwgs.User) (width 0.15))
+  (gr_line (start 248.285 73.66) (end 252.095 73.66) (layer Dwgs.User) (width 0.15))
   (gr_text 11/20 (at 241.935 76.073) (layer B.SilkS)
     (effects (font (size 1 1) (thickness 0.1)) (justify mirror))
@@
   )
   (dimension 43.18 (width 0.15) (layer Dwgs.User)
-    (gr_text "43.180 mm" (at 40.61 52.07 270) (layer Dwgs.User)
+    (gr_text "43.180 mm" (at 41.245 52.07 270) (layer Dwgs.User)
       (effects (font (size 1 1) (thickness 0.15)))
     )
-    (feature1 (pts (xy 54.61 73.66) (xy 41.323579 73.66)))
-    (feature2 (pts (xy 54.61 30.48) (xy 41.323579 30.48)))
-    (crossbar (pts (xy 41.91 30.48) (xy 41.91 73.66)))
-    (arrow1a (pts (xy 41.91 73.66) (xy 41.323579 72.533496)))
-    (arrow1b (pts (xy 41.91 73.66) (xy 42.496421 72.533496)))
-    (arrow2a (pts (xy 41.91 30.48) (xy 41.323579 31.606504)))
-    (arrow2b (pts (xy 41.91 30.48) (xy 42.496421 31.606504)))
+    (feature1 (pts (xy 58.42 73.66) (xy 41.958579 73.66)))
+    (feature2 (pts (xy 58.42 30.48) (xy 41.958579 30.48)))
+    (crossbar (pts (xy 42.545 30.48) (xy 42.545 73.66)))
+    (arrow1a (pts (xy 42.545 73.66) (xy 41.958579 72.533496)))
+    (arrow1b (pts (xy 42.545 73.66) (xy 43.131421 72.533496)))
+    (arrow2a (pts (xy 42.545 30.48) (xy 41.958579 31.606504)))
+    (arrow2b (pts (xy 42.545 30.48) (xy 43.131421 31.606504)))
   )
   (dimension 3.81 (width 0.15) (layer Dwgs.User)
@@
       (effects (font (size 1 1) (thickness 0.15)))
     )
-    (feature1 (pts (xy 54.61 26.67) (xy 38.783579 26.67)))
-    (feature2 (pts (xy 54.61 30.48) (xy 38.783579 30.48)))
+    (feature1 (pts (xy 58.42 26.67) (xy 38.783579 26.67)))
+    (feature2 (pts (xy 58.42 30.48) (xy 38.783579 30.48)))
     (crossbar (pts (xy 39.37 30.48) (xy 39.37 26.67)))
     (arrow1a (pts (xy 39.37 26.67) (xy 39.956421 27.796504)))
@@
       (effects (font (size 1 1) (thickness 0.15)))
     )
-    (feature1 (pts (xy 250.19 26.67) (xy 250.19 15.923579)))
-    (feature2 (pts (xy 58.42 26.67) (xy 58.42 15.923579)))
+    (feature1 (pts (xy 250.19 30.48) (xy 250.19 15.923579)))
+    (feature2 (pts (xy 58.42 30.48) (xy 58.42 15.923579)))
     (crossbar (pts (xy 58.42 16.51) (xy 250.19 16.51)))
     (arrow1a (pts (xy 250.19 16.51) (xy 249.063496 17.096421)))
@@
   (segment (start 58.42 30.48) (end 59.4142 30.48) (width 0.35) (layer B.Cu) (net 1))
   (segment (start 59.4142 30.48) (end 60.1171 29.7771) (width 0.35) (layer B.Cu) (net 1))
-  (segment (start 58.42 32.88) (end 58.42 71.26) (width 0.35) (layer B.Cu) (net 1))
   (segment (start 60.1171 72.9571) (end 60.1171 71.9629) (width 0.35) (layer B.Cu) (net 1))
   (segment (start 60.82 73.66) (end 60.1171 72.9571) (width 0.35) (layer B.Cu) (net 1))
@@
   (segment (start 249.348 73.66) (end 250.19 73.66) (width 0.35) (layer B.Cu) (net 1))
   (segment (start 244.268 68.58) (end 249.348 73.66) (width 0.35) (layer B.Cu) (net 1))
+  (segment (start 58.42 30.48) (end 58.42 46.99) (width 0.35) (layer B.Cu) (net 1))
+  (segment (start 58.42 46.99) (end 59.817 48.387) (width 0.35) (layer B.Cu) (net 1))
+  (segment (start 59.817 48.387) (end 59.817 50.546) (width 0.35) (layer B.Cu) (net 1))
+  (segment (start 59.817 50.546) (end 59.309 51.054) (width 0.35) (layer B.Cu) (net 1))
+  (segment (start 59.309 51.054) (end 59.309 54.229) (width 0.35) (layer B.Cu) (net 1))
+  (segment (start 59.309 54.229) (end 60.452 55.372) (width 0.35) (layer B.Cu) (net 1))
+  (segment (start 60.452 71.628) (end 58.42 73.66) (width 0.35) (layer B.Cu) (net 1))
+  (segment (start 60.452 55.372) (end 60.452 71.628) (width 0.35) (layer B.Cu) (net 1))
   (segment (start 111.0835 39.3708) (end 105.5077 39.3708) (width 0.35) (layer B.Cu) (net 2))
   (segment (start 105.5077 39.3708) (end 103.5051 37.3682) (width 0.35) (layer B.Cu) (net 2))
@@
   (segment (start 65.364001 43.220999) (end 65.2145 43.3705) (width 0.35) (layer F.Cu) (net 117))
   (segment (start 66.130999 72.299001) (end 67.31 71.12) (width 0.35) (layer B.Cu) (net 117))
-  (segment (start 60.161921 48.423079) (end 60.161921 69.116843) (width 0.35) (layer B.Cu) (net 117))
   (segment (start 63.344079 72.299001) (end 66.130999 72.299001) (width 0.35) (layer B.Cu) (net 117))
-  (segment (start 60.161921 69.116843) (end 63.344079 72.299001) (width 0.35) (layer B.Cu) (net 117))
-  (segment (start 64.135 44.45) (end 60.161921 48.423079) (width 0.35) (layer B.Cu) (net 117))
+  (segment (start 61.76299 70.717912) (end 63.344079 72.299001) (width 0.35) (layer B.Cu) (net 117))
+  (segment (start 61.76299 46.82201) (end 61.76299 70.717912) (width 0.35) (layer B.Cu) (net 117))
+  (segment (start 64.135 44.45) (end 61.76299 46.82201) (width 0.35) (layer B.Cu) (net 117))
   (segment (start 69.215 52.07) (end 70.3153 52.07) (width 0.2) (layer F.Cu) (net 118))
   (segment (start 77.56 53.67) (end 76.5097 53.67) (width 0.2) (layer F.Cu) (net 118))
